File: xc_nice_nano_tx_ board/xc_nice_nano_tx_ board.kicad_pcb (KiCad board)
At the start: 2 copper layers, 19.6 x 33 mm, 8 parts, among them J1 VibSensor, J2 BAT_MINUS_TAB, J3 BAT_PLUS_TAB, U1 nice_nano

Commit message: tweaked board. i think we're ready
Parts:
- moved C1 1.33 mm to (7.62, 6.10)
- moved C2 1.33 mm to (9.53, 6.10)
- moved J2 0.65 mm to (8.26, 9.65)
Connections:
- R1 pad 1: 3V3 -> BAT+
- U1 pad 18: unconnected-(U1-P0.29-LF-Pad18) -> P0.29
Routing:
- net BAT+: track 20.1 -> 39.7 mm
- net 3V3: track 14.7 -> 0.00 mm
- net BAT-: track 63.1 -> 56.9 mm
- added copper zone on B.Cu, net BAT-
Other:
- board size 19.6 x 33 mm -> 25.3 x 33 mm
