File: xc_nice_nano_tx_ board/xc_nice_nano_tx_ board.kicad_sch (KiCad schematic)
At the start: 10 parts, among them J1 VibSensor, J2 BAT_MINUS_TAB, J3 BAT_PLUS_TAB, U1 nice_nano

Commit message: tweaked board. i think we're ready
Parts:
- removed R2, R3: 470k, symbol Device:R
